Commit message: Increasing robot model size in simulation.
This reduces robot bouncing when colliding.

File: software/model/unball_robot.urdf (robot description, URDF)
Before this commit: robot test_robot, 3 links, 2 joints
Links:
- link base_link: geometry collision box size=0.075 0.075 0.095; visual box size=0.075 0.075 0.095
